File: Power/power_board2_v2.0.sch (EAGLE design)
At the start: 58 parts, among them J0_PLOAD_CONN 172648-0102, J1_B3_CONN 105313-1102, J2_LORA_CONN 105313-1102, J3_SPOT_CONN 105313-1102, J4_SSSBOARD_CONN 172648-0102, Q1 FQD11P06TM

Commit message: Included larger size mounting holes on both .brd files, pretty much finished board 2 (haven't GND'ed yet, need a design review)
Parts:
- removed B3_VOLT_REG, LORA_VOLT_REG, SPOT_VOLT_REG: LT3681, linear-technology:LT3681
- removed INDUCTOR_3: CDRH104RNP-150NC, CDRH104RNP-150NC:CDRH104RNP-150NC
- removed J0_PLOAD_CONN, J4_SSSBOARD_CONN: 172648-0102, 172648-0102:172648-0102
- removed J1_B3_CONN, J2_LORA_CONN, J3_SPOT_CONN: 105313-1102, 105313-1102:105313-1102
- removed L4, L5: SBC2-6R8-242, SBC2-6R8-242:SBC2-6R8-242
- removed Q1: FQD11P06TM, FQD11P06TM:FQD11P06TM
- removed R39: 0, rcl:R-US_0207/2V
- removed XL6009_BOOST_CONV_DAUGHTERBOARD: CP8-ADJ, userlib:CP8-ADJ
- added 12VNO1_VOLT_REG, 12VNO2_VOLT_REG, 5VNO1_VOLT_REG, 5VNO2_VOLT_REG, 9VNO1_VOLT_REG, 9VNO2_VOLT_REG: LT3681, linear-technology:LT3681
- added C10, C16, C59: 100n, 06031C104KAT2A:06031C104KAT2A
- added C11, C17, C28: .33n, 08053C334KAT2A:08053C334KAT2A
- added C13, C26, C58: 10u, 22201C106KAT2A:22201C106KAT2A
- added C14, C18, C29, C36: 220n, 08051C224KAT2A:08051C224KAT2A
- added C19: 26.7u, 12103C226KAT2A:12103C226KAT2A
- added C20, C21, C25: 470n, 06033C474JAT2A:06033C474JAT2A
- added C60, C61, C62, C63: 100n, 06033C104KAT4A:06033C104KAT4A
- added INDUCTOR_2, INDUCTOR_4, INDUCTOR_5, INDUCTOR_6, INDUCTOR_7, INDUCTOR_8: CDRH104RNP-150NC, CDRH104RNP-150NC:CDRH104RNP-150NC
- added J0_VLINE_CONN: 172648-0102, 172648-0102:172648-0102
- added J1_5VNO1_CONN, J2_5VNO2_CONN: 105313-1102, 105313-1102:105313-1102
- added J3_9VNO1_CONN, J4_9VNO2_CONN: 43650-0212, 43650-0212:43650-0212
- added J5_12VNO1_CONN, J6_12VNO2_CONN: 87427-0212, 87427-0212:87427-0212
- added Q2: FQD11P06TM, FQD11P06TM:FQD11P06TM
- added R23: 845k, rcl:R-US_R0603
- added R24, R27, R31, R34, R64, R65, R69: 0, rcl:R-US_0207/2V
- added R25: 100k, rcl:R-US_R0603
- added R28, R32, R35, R61: 133k, rcl:R-US_R0603
- added R29, R36, R62: 20k, rcl:R-US_R0603
- added R30, R68: 15k, rcl:R-US_R0603
- added R33: 590k, rcl:R-US_R0603
- added R63: 806k, rcl:R-US_R0603
- C1, C5: value 100n -> 10u; device 06033C104KAT4A:06033C104KAT4A -> 22201C106KAT2A:22201C106KAT2A
- C12: value 50.8u -> 220n; device 12103C226KAT2A:12103C226KAT2A -> 08051C224KAT2A:08051C224KAT2A
- C2: value 470n -> 100n; device 06033C474JAT2A:06033C474JAT2A -> 06031C104KAT2A:06031C104KAT2A
- C22: value .33n -> 26.7u; device 08053C334KAT2A:08053C334KAT2A -> 12103C226KAT2A:12103C226KAT2A
- C23: value .33n -> 470n; device 08053C334KAT2A:08053C334KAT2A -> 06033C474JAT2A:06033C474JAT2A
- C24: value .33n -> 22u; device 08053C334KAT2A:08053C334KAT2A -> 12103C226KAT2A:12103C226KAT2A
- C27: value 50.8u -> 100n; device 12103C226KAT2A:12103C226KAT2A -> 06031C104KAT2A:06031C104KAT2A
- C3, C4: value 470n -> .33n; device 06033C474JAT2A:06033C474JAT2A -> 08053C334KAT2A:08053C334KAT2A
- C30: value 220n -> 10u; device 08051C224KAT2A:08051C224KAT2A -> 22201C106KAT2A:22201C106KAT2A
- C31: value 220n -> 100n; device 08051C224KAT2A:08051C224KAT2A -> 06031C104KAT2A:06031C104KAT2A
- C32: value 220n -> 22u; device 08051C224KAT2A:08051C224KAT2A -> 12103C226KAT2A:12103C226KAT2A
- C33: value 10u -> 470n; device 22201C106KAT2A:22201C106KAT2A -> 06033C474JAT2A:06033C474JAT2A
- C34: value 10u -> 100n; device 22201C106KAT2A:22201C106KAT2A -> 06033C104KAT4A:06033C104KAT4A
- C35: value 10u -> .33n; device 22201C106KAT2A:22201C106KAT2A -> 08053C334KAT2A:08053C334KAT2A
- C6: value 100n -> 220n; device 06033C104KAT4A:06033C104KAT4A -> 08051C224KAT2A:08051C224KAT2A
- C7: value 100n -> 50.8u; device 06031C104KAT2A:06031C104KAT2A -> 12103C226KAT2A:12103C226KAT2A
- C8: value 100n -> 470n; device 06031C104KAT2A:06031C104KAT2A -> 06033C474JAT2A:06033C474JAT2A
- C9: device 06031C104KAT2A:06031C104KAT2A -> 06033C104KAT4A:06033C104KAT4A
- R1: value 0 -> 133k; device rcl:R-US_0207/2V -> rcl:R-US_R0603; DESC RES SMD 10K OHM 1% 1/8W 0805 -> (none); MFR Yageo -> (none); MPN RC0805FR-0710KL -> (none)
- R10: value 133k -> 20k
- R11: value 20k -> 15k
- R12: value 200k -> 0; device rcl:R-US_R0603 -> rcl:R-US_0207/2V; DESC (none) -> RES SMD 10K OHM 1% 1/8W 0805; MFR (none) -> Yageo; MPN (none) -> RC0805FR-0710KL
- R13: value 590k -> 133k
- R15: value 0 -> 200k; device rcl:R-US_0207/2V -> rcl:R-US_R0603; DESC RES SMD 10K OHM 1% 1/8W 0805 -> (none); MFR Yageo -> (none); MPN RC0805FR-0710KL -> (none)
- R16: value 0 -> 20k; device rcl:R-US_0207/2V -> rcl:R-US_R0603; DESC RES SMD 10K OHM 1% 1/8W 0805 -> (none); MFR Yageo -> (none); MPN RC0805FR-0710KL -> (none)
- R18: value 15k -> 0; device rcl:R-US_R0603 -> rcl:R-US_0207/2V; DESC (none) -> RES SMD 10K OHM 1% 1/8W 0805; MFR (none) -> Yageo; MPN (none) -> RC0805FR-0710KL
- R19: value 15k -> 133k
- R20: value 0 -> 806k; device rcl:R-US_0207/2V -> rcl:R-US_R0603; DESC RES SMD 10K OHM 1% 1/8W 0805 -> (none); MFR Yageo -> (none); MPN RC0805FR-0710KL -> (none)
- R22: value 0 -> 100k; device rcl:R-US_0207/2V -> rcl:R-US_R0603; DESC RES SMD 10K OHM 1% 1/8W 0805 -> (none); MFR Yageo -> (none); MPN RC0805FR-0710KL -> (none)
- R26: value 0 -> 845k; device rcl:R-US_0207/2V -> rcl:R-US_R0603; DESC RES SMD 10K OHM 1% 1/8W 0805 -> (none); MFR Yageo -> (none); MPN RC0805FR-0710KL -> (none)
- R4: value 200k -> 15k
- R5: value 590k -> 0; device rcl:R-US_R0603 -> rcl:R-US_0207/2V; DESC (none) -> RES SMD 10K OHM 1% 1/8W 0805; MFR (none) -> Yageo; MPN (none) -> RC0805FR-0710KL
- R6: value 133k -> 15k
- R7: value 20k -> 0; device rcl:R-US_R0603 -> rcl:R-US_0207/2V; DESC (none) -> RES SMD 10K OHM 1% 1/8W 0805; MFR (none) -> Yageo; MPN (none) -> RC0805FR-0710KL
Connections:
- removed net CBOOST_B3: B3_VOLT_REG.BOOST, C2.1
- removed net CBOOST_LORA: C3.1, LORA_VOLT_REG.BOOST
- removed net CBOOST_SPOT: C4.1, SPOT_VOLT_REG.BOOST
- removed net FB_B3: B3_VOLT_REG.FB, R8.2, R9.2
- removed net FB_LORA: LORA_VOLT_REG.FB, R4.2, R5.2
- removed net FB_SPOT: R12.2, R13.2, SPOT_VOLT_REG.FB
- removed net N$2: C23.1, R3.1
- removed net RT_B3: B3_VOLT_REG.RT, R6.2
- removed net RT_LORA: LORA_VOLT_REG.RT, R2.2
- removed net RT_SPOT: R10.2, SPOT_VOLT_REG.RT
- removed net RUN/SS_B3: B3_VOLT_REG.RUN/SS, C30.1, R17.1
- removed net RUN/SS_LORA: C31.1, LORA_VOLT_REG.RUN/SS, R18.1
- removed net RUN/SS_SPOT: C32.1, R19.1, SPOT_VOLT_REG.RUN/SS
- removed net SW_B3: B3_VOLT_REG.DC, B3_VOLT_REG.DC@1, B3_VOLT_REG.SW, C2.2, INDUCTOR_3.1
- removed net SW_LORA: C3.2, L5.1, LORA_VOLT_REG.DC, LORA_VOLT_REG.DC@1, LORA_VOLT_REG.SW
- removed net SW_SPOT: C4.2, L4.1, SPOT_VOLT_REG.DC, SPOT_VOLT_REG.DC@1, SPOT_VOLT_REG.SW
- removed net VC_B3: B3_VOLT_REG.VC, R7.2
- removed net VC_LORA: LORA_VOLT_REG.VC, R3.2
- removed net VC_SPOT: R11.2, SPOT_VOLT_REG.VC
- removed net VIN_B3: B3_VOLT_REG.VIN, C33.1, C7.1, R17.2, R39.1
- removed net VIN_LORA: C34.1, C8.1, LORA_VOLT_REG.VIN, R1.1, R18.2
- removed net VIN_SPOT: C35.1, C9.1, R14.1, R19.2, SPOT_VOLT_REG.VIN
- removed net VIN_XL6009: R15.1, XL6009_BOOST_CONV_DAUGHTERBOARD.IN+
- removed net V_B3: B3_VOLT_REG.BD, B3_VOLT_REG.BIAS, C1.1, C15.1, INDUCTOR_3.2, R16.2, R9.1
- removed net V_B31: J1_B3_CONN.1, R16.1
- removed net V_LORA: C27.1, C5.1, L5.2, LORA_VOLT_REG.BD, LORA_VOLT_REG.BIAS, R20.2, R5.1
- removed net V_LORA1: J2_LORA_CONN.1, R20.1
- removed net V_PLOAD: Q1.S, R1.2, R14.2, R15.2, R39.2
- removed net V_PLOAD0: Q1.D, R26.1
- removed net V_PLOAD00: J0_PLOAD_CONN.2, R26.2
- removed net V_SPOT: C12.1, C6.1, L4.2, R13.1, R21.2, SPOT_VOLT_REG.BD, SPOT_VOLT_REG.BIAS
- removed net V_SPOT1: J3_SPOT_CONN.1, R21.1
- removed net V_SSS: R22.2, XL6009_BOOST_CONV_DAUGHTERBOARD.OUT+
- removed net V_SSS1: J4_SSSBOARD_CONN.1, R22.1
- new net CBOOST_12VNO1: 12VNO1_VOLT_REG.BOOST, C23.1
- new net CBOOST_12VNO2: 12VNO2_VOLT_REG.BOOST, C25.1
- new net CBOOST_5VNO1: 5VNO1_VOLT_REG.BOOST, C8.1
- new net CBOOST_5VNO2: 5VNO2_VOLT_REG.BOOST, C33.1
- new net CBOOST_9VNO1: 9VNO1_VOLT_REG.BOOST, C20.1
- new net CBOOST_9VNO2: 9VNO2_VOLT_REG.BOOST, C21.1
- new net FB_12VNO1: 12VNO1_VOLT_REG.FB, R22.2, R23.2
- new net FB_12VNO2: 12VNO2_VOLT_REG.FB, R25.2, R26.2
- new net FB_5VNO1: 5VNO1_VOLT_REG.FB, R8.2, R9.2
- new net FB_5VNO2: 5VNO2_VOLT_REG.FB, R15.2, R33.2
- new net FB_9VNO1: 9VNO1_VOLT_REG.FB, R19.2, R20.2
- new net FB_9VNO2: 9VNO2_VOLT_REG.FB, R32.2, R63.2
- new net N$17: C28.1, R29.1
- new net N$18: C35.1, R36.1
- new net N$5: C11.1, R10.1
- new net N$6: C17.1, R16.1
- new net RT_12VNO1: 12VNO1_VOLT_REG.RT, R28.2
- new net RT_12VNO2: 12VNO2_VOLT_REG.RT, R35.2
- new net RT_5VNO1: 5VNO1_VOLT_REG.RT, R61.2
- new net RT_5VNO2: 5VNO2_VOLT_REG.RT, R2.2
- new net RT_9VNO1: 9VNO1_VOLT_REG.RT, R1.2
- new net RT_9VNO2: 9VNO2_VOLT_REG.RT, R13.2
- new net RUN/SS_12VNO1: 12VNO1_VOLT_REG.RUN/SS, C29.1, R30.1
- new net RUN/SS_12VNO2: 12VNO2_VOLT_REG.RUN/SS, C36.1, R68.1
- new net RUN/SS_5VNO1: 5VNO1_VOLT_REG.RUN/SS, C6.1, R6.1
- new net RUN/SS_5VNO2: 5VNO2_VOLT_REG.RUN/SS, C14.1, R4.1
- new net RUN/SS_9VNO1: 9VNO1_VOLT_REG.RUN/SS, C12.1, R11.1
- new net RUN/SS_9VNO2: 9VNO2_VOLT_REG.RUN/SS, C18.1, R17.1
- new net SW_12VNO1: 12VNO1_VOLT_REG.DC, 12VNO1_VOLT_REG.DC@1, 12VNO1_VOLT_REG.SW, C23.2, INDUCTOR_7.1
- new net SW_12VNO2: 12VNO2_VOLT_REG.DC, 12VNO2_VOLT_REG.DC@1, 12VNO2_VOLT_REG.SW, C25.2, INDUCTOR_8.1
- new net SW_5VNO1: 5VNO1_VOLT_REG.DC, 5VNO1_VOLT_REG.DC@1, 5VNO1_VOLT_REG.SW, C8.2, INDUCTOR_2.1
- new net SW_5VNO2: 5VNO2_VOLT_REG.DC, 5VNO2_VOLT_REG.DC@1, 5VNO2_VOLT_REG.SW, C33.2, INDUCTOR_4.1
- new net SW_9VNO1: 9VNO1_VOLT_REG.DC, 9VNO1_VOLT_REG.DC@1, 9VNO1_VOLT_REG.SW, C20.2, INDUCTOR_5.1
- new net SW_9VNO2: 9VNO2_VOLT_REG.DC, 9VNO2_VOLT_REG.DC@1, 9VNO2_VOLT_REG.SW, C21.2, INDUCTOR_6.1
- new net VC_12VNO1: 12VNO1_VOLT_REG.VC, R29.2
- new net VC_12VNO2: 12VNO2_VOLT_REG.VC, R36.2
- new net VC_5VNO1: 5VNO1_VOLT_REG.VC, R62.2
- new net VC_5VNO2: 5VNO2_VOLT_REG.VC, R3.2
- new net VC_9VNO1: 9VNO1_VOLT_REG.VC, R10.2
- new net VC_9VNO2: 9VNO2_VOLT_REG.VC, R16.2
- new net VIN_12VNO1: 12VNO1_VOLT_REG.VIN, C26.1, C27.1, R30.2, R31.1
- new net VIN_12VNO2: 12VNO2_VOLT_REG.VIN, C30.1, C31.1, R68.2, R69.1
- new net VIN_5VNO1: 5VNO1_VOLT_REG.VIN, C58.1, C59.1, R6.2, R7.1
- new net VIN_5VNO2: 5VNO2_VOLT_REG.VIN, C1.1, C2.1, R4.2, R5.1
- new net VIN_9VNO1: 9VNO1_VOLT_REG.VIN, C10.1, C5.1, R11.2, R12.1
- new net VIN_9VNO2: 9VNO2_VOLT_REG.VIN, C13.1, C16.1, R17.2, R18.1
- new net V_12VNO1: 12VNO1_VOLT_REG.BD, 12VNO1_VOLT_REG.BIAS, C24.1, C63.1, INDUCTOR_7.2, R23.1, R24.2
- new net V_12VNO1_0: J5_12VNO1_CONN.2, R24.1
- new net V_12VNO2: 12VNO2_VOLT_REG.BD, 12VNO2_VOLT_REG.BIAS, C32.1, C62.1, INDUCTOR_8.2, R26.1, R27.2
- new net V_12VNO2_0: J6_12VNO2_CONN.2, R27.1
- new net V_5VNO1: 5VNO1_VOLT_REG.BD, 5VNO1_VOLT_REG.BIAS, C7.1, C9.1, INDUCTOR_2.2, R14.2, R9.1
- new net V_5VNO1_0: J1_5VNO1_CONN.1, R14.1
- new net V_5VNO2: 5VNO2_VOLT_REG.BD, 5VNO2_VOLT_REG.BIAS, C15.1, C34.1, INDUCTOR_4.2, R33.1, R34.2
- new net V_5VNO2_0: J2_5VNO2_CONN.1, R34.1
- new net V_9VNO1: 9VNO1_VOLT_REG.BD, 9VNO1_VOLT_REG.BIAS, C19.1, C60.1, INDUCTOR_5.2, R20.1, R21.2
- new net V_9VNO1_0: J3_9VNO1_CONN.1, R21.1
- new net V_9VNO2: 9VNO2_VOLT_REG.BD, 9VNO2_VOLT_REG.BIAS, C22.1, C61.1, INDUCTOR_6.2, R63.1, R64.2
- new net V_9VNO2_0: J4_9VNO2_CONN.1, R64.1
- new net V_VLINE: Q2.S, R12.2, R18.2, R31.2, R5.2, R69.2, R7.2
- new net V_VLINE0: Q2.D, R65.1
- new net V_VLINE00: J0_VLINE_CONN.2, R65.2
- net GND: now also 12VNO1_VOLT_REG.DA, 12VNO1_VOLT_REG.GND, 12VNO1_VOLT_REG.GND@1, 12VNO1_VOLT_REG.GND@2, 12VNO2_VOLT_REG.GND, 12VNO2_VOLT_REG.GND@1, 12VNO2_VOLT_REG.GND@2, 5VNO1_VOLT_REG.DA, 5VNO1_VOLT_REG.GND, 5VNO1_VOLT_REG.GND@1, 5VNO1_VOLT_REG.GND@2, 5VNO2_VOLT_REG.DA, 5VNO2_VOLT_REG.GND, 5VNO2_VOLT_REG.GND@1, 5VNO2_VOLT_REG.GND@2, 9VNO1_VOLT_REG.DA, 9VNO1_VOLT_REG.GND, 9VNO1_VOLT_REG.GND@1, 9VNO1_VOLT_REG.GND@2, 9VNO2_VOLT_REG.DA, 9VNO2_VOLT_REG.GND, 9VNO2_VOLT_REG.GND@1, 9VNO2_VOLT_REG.GND@2, C10.2, C11.2, C13.2, C14.2, C16.2, C17.2, C18.2, C19.2, C2.2, C26.2, C28.2, C29.2, C3.2, C36.2, C4.2, C58.2, C59.2, C60.2, C61.2, C62.2, C63.2, J0_VLINE_CONN.1, J1_5VNO1_CONN.2, J2_5VNO2_CONN.2, J3_9VNO1_CONN.2, J4_9VNO2_CONN.2, J5_12VNO1_CONN.1, J6_12VNO2_CONN.1, Q2.G, R1.1, R13.1, R15.1, R19.1, R22.1, R25.1, R28.1, R32.1, R35.1, R61.1; no longer B3_VOLT_REG.DA, B3_VOLT_REG.GND, B3_VOLT_REG.GND@1, B3_VOLT_REG.GND@2, C23.2, C33.2, C8.2, J0_PLOAD_CONN.1, J1_B3_CONN.2, J2_LORA_CONN.2, J3_SPOT_CONN.2, J4_SSSBOARD_CONN.2, LORA_VOLT_REG.DA, LORA_VOLT_REG.GND, LORA_VOLT_REG.GND@1, LORA_VOLT_REG.GND@2, Q1.G, R10.1, R12.1, R4.1, R6.1, SPOT_VOLT_REG.DA, SPOT_VOLT_REG.GND, SPOT_VOLT_REG.GND@1, SPOT_VOLT_REG.GND@2, XL6009_BOOST_CONV_DAUGHTERBOARD.IN-, XL6009_BOOST_CONV_DAUGHTERBOARD.OUT-
- net N$1: now also C4.1, R62.1; no longer C22.1, R7.1
- net N$4: now also C3.1, R3.1; no longer C24.1, R11.1
Other:
- note added: "10uH"
- note added: "12V"
- note added: "1x22uF and 1x4.7uF caps to be stacked vertically"
- note added: "22u"
- note added: "26.7u"
- note added: "5V/9V/12V Voltage Line Power Board"
- note added: "7uH"
- note added: "9V"
- note added: "Connector "J0_VLINE_CONN" brings in the voltage line(s) power from the "J3 Pload" connector on the AUV's existing Power Controller Board"
- note added: "Connector "J1_5VNO1_CONN" is a 5V voltage line output"
- note added: "Connector "J2_5VNO2_CONN" is a 5V voltage line output"
- note added: "Connector "J3_9VNO1_CONN" is a 9V voltage line output"
- note added: "Connector "J4_9VNO2_CONN" is a 9V voltage line output"
- note added: "Connector "J5_12VNO1_CONN" is a 12V voltage line output"
- note added: "Connector "J6_12VNO2_CONN" is a 12V voltage line output"
- note added: "J1_5VNO1_CONN"
- note added: "J2_5VNO2_CONN"
- note removed: "220n"
- note removed: "24V"
- note removed: "470n"
- note removed: "6.8uH"
- note removed: "Connector "J0_PLOAD_CONN" brings in the payload power from the "J3 Pload" connector on the AUV's existing Power Controller Board"
- note removed: "Connector "J1_B3_CONN" powers the Payload's BeagleBone Black uprocessor"
- note removed: "Connector "J2_LORA_CONN" powers the Adafruit Feather M0 with RFM95 LoRa Radio communication device."
- note removed: "Connector "J3_SPOT_CONN" powers the SPOT Trace beacon emergency location device."
- note removed: "Connector "J4_SSSBOARD_CONN" powers the Imagenex Ethernet Sidescan Sonar board."
- note removed: "Payload Power Board"
- note removed: "XL6009_BOOST_CONV_DAUGHTERBOARD"
- moved on the sheet: C1, C12, C15, C2, C22, C23, C24, C27, C3, C30, C31, C32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
